File: schematics/board_connector.kicad_sch (KiCad schematic)
At the start: 1 part, among them J2 Conn_02x20_Odd_Even

Commit message: kicad: Run Assign footprint
Parts:
- J2: footprint (none) -> Connector_PinHeader_2.54mm:PinHeader_2x20_P2.54mm_Vertical
Connections:
- net TURN_L_N: now reaches J2.16 (Pin_16)
- net TURN_R_N: now reaches J2.20 (Pin_20)
- no-connect marks 17 -> 15
Changed lines of the file:
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@@
 	)
 	(junction
-		(at 109.22 90.17)
+		(at 96.52 90.17)
 		(diameter 0)
 		(color 0 0 0 0)
@@
 	)
 	(no_connect
+		(at 134.62 97.79)
+	)
+	(no_connect
+		(at 134.62 72.39)
+	)
+	(no_connect
+		(at 147.32 90.17)
+	)
+	(no_connect
+		(at 134.62 95.25)
+	)
+	(no_connect
 		(at 134.62 74.93)
 	)
 	(no_connect
-		(at 134.62 97.79)
-	)
-	(no_connect
-		(at 134.62 72.39)
-	)
-	(no_connect
-		(at 147.32 90.17)
-	)
-	(no_connect
-		(at 134.62 95.25)
-	)
-	(no_connect
 		(at 147.32 92.71)
 	)
@@
 	)
 	(no_connect
-		(at 134.62 77.47)
-	)
-	(no_connect
 		(at 134.62 92.71)
 	)
@@
 	)
 	(no_connect
-		(at 134.62 82.55)
-	)
-	(no_connect
 		(at 147.32 87.63)
 	)
 	(wire
 		(pts
-			(xy 109.22 69.85) (xy 134.62 69.85)
+			(xy 96.52 69.85) (xy 134.62 69.85)
 		)
 		(stroke
@@
 	(wire
 		(pts
-			(xy 109.22 90.17) (xy 109.22 121.92)
+			(xy 96.52 90.17) (xy 96.52 121.92)
 		)
 		(stroke
@@
 	(wire
 		(pts
-			(xy 109.22 69.85) (xy 109.22 90.17)
+			(xy 96.52 69.85) (xy 96.52 90.17)
 		)
 		(stroke
@@
 	(wire
 		(pts
-			(xy 109.22 121.92) (xy 130.81 121.92)
+			(xy 96.52 121.92) (xy 130.81 121.92)
 		)
 		(stroke
@@
 	(wire
 		(pts
+			(xy 132.08 77.47) (xy 134.62 77.47)
+		)
+		(stroke
+			(width 0)
+			(type default)
+		)
+	)
+	(wire
+		(pts
 			(xy 177.8 74.93) (xy 177.8 82.55)
 		)
@@
 	(wire
 		(pts
+			(xy 120.65 82.55) (xy 134.62 82.55)
+		)
+		(stroke
+			(width 0)
+			(type default)
+		)
+	)
+	(wire
+		(pts
 			(xy 106.68 59.69) (xy 115.57 59.69)
 		)
@@
 	(wire
 		(pts
+			(xy 96.52 90.17) (xy 134.62 90.17)
+		)
+		(stroke
+			(width 0)
+			(type default)
+		)
+	)
+	(wire
+		(pts
 			(xy 120.65 105.41) (xy 134.62 105.41)
-		)
-		(stroke
-			(width 0)
-			(type default)
-		)
-	)
-	(wire
-		(pts
-			(xy 109.22 90.17) (xy 134.62 90.17)
 		)
 		(stroke
@@
 				)
 				(justify left)
+			)
+		)
+	)
+	(global_label "TURN_L_N"
+		(shape input)
+		(at 132.08 77.47 180)
+		(fields_autoplaced yes)
+		(effects
+			(font
+				(size 1.27 1.27)
+			)
+			(justify right)
+		)
+		(property "Intersheetrefs" "${INTERSHEET_REFS}"
+			(at 119.9024 77.47 0)
+			(hide yes)
+			(show_name no)
+			(do_not_autoplace no)
+			(effects
+				(font
+					(size 1.27 1.27)
+				)
+				(justify right)
+			)
+		)
+	)
+	(global_label "TURN_R_N"
+		(shape input)
+		(at 120.65 82.55 180)
+		(fields_autoplaced yes)
+		(effects
+			(font
+				(size 1.27 1.27)
+			)
+			(justify right)
+		)
+		(property "Intersheetrefs" "${INTERSHEET_REFS}"
+			(at 108.2305 82.55 0)
+			(hide yes)
+			(show_name no)
+			(do_not_autoplace no)
+			(effects
+				(font
+					(size 1.27 1.27)
+				)
+				(justify right)
 			)
 		)
@@
 			)
 		)
-		(property "Footprint" ""
+		(property "Footprint" "Connector_PinHeader_2.54mm:PinHeader_2x20_P2.54mm_Vertical"
 			(at 142.24 82.55 0)
 			(hide yes)

Commit message: schematics: Add mounting points for the PCB
Parts:
- added H1, H2, H3, H4: MountingHole_Pad, symbol Mechanical:MountingHole_Pad
- J2: value Conn_02x20_Odd_Even -> BOARD
Connections:
- net ENC_B: now also J2.32 (Pin_32); no longer J2.38 (Pin_38)
- net GND: now also H1.1, H2.1, H3.1, H4.1
Other:
- note added: "TP_INT via bodge wire TP2"
