File: schematics/buzzer_motor.kicad_sch (KiCad schematic)
At the start: 11 parts, among them J6 Conn_01x04, Q1 AO3400A, Q2 AO3400A

Commit message: kicad: Run Assign footprint
Parts:
- C10, C11: footprint (none) -> Capacitor_SMD:C_0805_2012Metric
- J6: footprint (none) -> Connector_JST:JST_XH_B4B-XH-A_1x04_P2.50mm_Vertical
- R12, R13, R14, R15: footprint (none) -> Resistor_SMD:R_0805_2012Metric
Changed lines of the file:
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@@
 			)
 		)
-		(property "Footprint" ""
+		(property "Footprint" "Resistor_SMD:R_0805_2012Metric"
 			(at 83.312 165.1 90)
 			(hide yes)
@@
 			)
 		)
-		(property "Footprint" ""
+		(property "Footprint" "Capacitor_SMD:C_0805_2012Metric"
 			(at 59.3852 135.89 0)
 			(hide yes)
@@
 			)
 		)
-		(property "Footprint" ""
+		(property "Footprint" "Resistor_SMD:R_0805_2012Metric"
 			(at 83.312 82.55 90)
 			(hide yes)
@@
 			)
 		)
-		(property "Footprint" ""
+		(property "Footprint" "Capacitor_SMD:C_0805_2012Metric"
 			(at 59.3852 53.34 0)
 			(hide yes)
@@
 			)
 		)
-		(property "Footprint" ""
+		(property "Footprint" "Connector_JST:JST_XH_B4B-XH-A_1x04_P2.50mm_Vertical"
 			(at 177.8 39.37 0)
 			(hide yes)
@@
 			)
 		)
-		(property "Footprint" ""
+		(property "Footprint" "Resistor_SMD:R_0805_2012Metric"
 			(at 97.282 71.12 90)
 			(hide yes)
@@
 			)
 		)
-		(property "Footprint" ""
+		(property "Footprint" "Resistor_SMD:R_0805_2012Metric"
 			(at 97.282 153.67 90)
 			(hide yes)

Commit message: schematics: Add mounting points for the PCB
Parts:
- J6: value Conn_01x04 -> MOTOR
Connections:
- net MOTOR_R_N: now reaches C11.2, D6.2 (A), J6.4 (Pin_4), Q2.3 (D)
- net MOTOR_L_N: now reaches C10.2, D5.2 (A), J6.2 (Pin_2), Q1.3 (D)
Changed lines of the file:
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@@
+	)
+	(junction
+		(at 116.84 121.92)
+		(diameter 0)
+		(color 0 0 0 0)
+	)
+	(junction
+		(at 113.03 39.37)
+		(diameter 0)
+		(color 0 0 0 0)
 	)
 	(junction
@@
 	(wire
 		(pts
-			(xy 76.2 121.92) (xy 148.59 121.92)
+			(xy 76.2 121.92) (xy 116.84 121.92)
 		)
 		(stroke
@@
 	(wire
 		(pts
+			(xy 113.03 39.37) (xy 172.72 39.37)
+		)
+		(stroke
+			(width 0)
+			(type default)
+		)
+	)
+	(wire
+		(pts
+			(xy 113.03 39.37) (xy 113.03 41.91)
+		)
+		(stroke
+			(width 0)
+			(type default)
+		)
+	)
+	(wire
+		(pts
 			(xy 99.06 144.78) (xy 99.06 149.86)
 		)
@@
 	(wire
 		(pts
-			(xy 76.2 39.37) (xy 172.72 39.37)
+			(xy 76.2 39.37) (xy 113.03 39.37)
 		)
 		(stroke
@@
 	(wire
 		(pts
+			(xy 116.84 121.92) (xy 148.59 121.92)
+		)
+		(stroke
+			(width 0)
+			(type default)
+		)
+	)
+	(wire
+		(pts
+			(xy 116.84 121.92) (xy 116.84 125.73)
+		)
+		(stroke
+			(width 0)
+			(type default)
+		)
+	)
+	(wire
+		(pts
 			(xy 34.29 144.78) (xy 34.29 135.89)
 		)
@@
 			(width 0)
 			(type default)
+		)
+	)
+	(label "MOTOR_L_N"
+		(at 113.03 41.91 270)
+		(effects
+			(font
+				(size 1.27 1.27)
+			)
+			(justify right bottom)
+		)
+	)
+	(label "MOTOR_R_N"
+		(at 116.84 125.73 270)
+		(effects
+			(font
+				(size 1.27 1.27)
+			)
+			(justify right bottom)
 		)
 	)
@@
 			)
 		)
-		(property "Value" "Conn_01x04"
+		(property "Value" "MOTOR"
 			(at 177.8 33.02 0)
 			(show_name no)
