File: schematics/indicators.kicad_sch (KiCad schematic)
At the start: 7 parts, among them J7 Conn_01x04, Q3 AO3400A, Q4 AO3400A

Commit message: kicad: Run Assign footprint
Parts:
- J7: footprint (none) -> Connector_JST:JST_XH_B4B-XH-A_1x04_P2.50mm_Vertical
- R16, R17, R18, R19: footprint (none) -> Resistor_SMD:R_0805_2012Metric
Changed lines of the file:
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@@
 			)
 		)
-		(property "Footprint" ""
+		(property "Footprint" "Resistor_SMD:R_0805_2012Metric"
 			(at 82.042 156.21 90)
 			(hide yes)
@@
 			)
 		)
-		(property "Footprint" ""
+		(property "Footprint" "Connector_JST:JST_XH_B4B-XH-A_1x04_P2.50mm_Vertical"
 			(at 143.51 39.37 0)
 			(hide yes)
@@
 			)
 		)
-		(property "Footprint" ""
+		(property "Footprint" "Resistor_SMD:R_0805_2012Metric"
 			(at 96.012 144.78 90)
 			(hide yes)
@@
 			)
 		)
-		(property "Footprint" ""
+		(property "Footprint" "Resistor_SMD:R_0805_2012Metric"
 			(at 82.042 80.01 90)
 			(hide yes)
@@
 			)
 		)
-		(property "Footprint" ""
+		(property "Footprint" "Resistor_SMD:R_0805_2012Metric"
 			(at 96.012 68.58 90)
 			(hide yes)

Commit message: schematics: Add mounting points for the PCB
Parts:
- J7: value Conn_01x04 -> IND_OUTPUT
Connections:
- net LAMP_L_N: now reaches J7.2 (Pin_2), Q3.3 (D)
- net LAMP_R_N: now reaches J7.4 (Pin_4), Q4.3 (D)
Changed lines of the file:
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@@
+	)
+	(junction
+		(at 92.71 39.37)
+		(diameter 0)
+		(color 0 0 0 0)
 	)
 	(junction
@@
 		(color 0 0 0 0)
 	)
+	(junction
+		(at 119.38 115.57)
+		(diameter 0)
+		(color 0 0 0 0)
+	)
 	(wire
 		(pts
@@
 	(wire
 		(pts
-			(xy 72.39 39.37) (xy 138.43 39.37)
+			(xy 72.39 39.37) (xy 92.71 39.37)
 		)
 		(stroke
@@
 	(wire
 		(pts
+			(xy 119.38 113.03) (xy 119.38 115.57)
+		)
+		(stroke
+			(width 0)
+			(type default)
+		)
+	)
+	(wire
+		(pts
 			(xy 72.39 39.37) (xy 72.39 59.69)
 		)
@@
 	(wire
 		(pts
-			(xy 72.39 115.57) (xy 134.62 115.57)
+			(xy 72.39 115.57) (xy 119.38 115.57)
 		)
 		(stroke
@@
 	(wire
 		(pts
+			(xy 119.38 115.57) (xy 134.62 115.57)
+		)
+		(stroke
+			(width 0)
+			(type default)
+		)
+	)
+	(wire
+		(pts
 			(xy 72.39 115.57) (xy 72.39 135.89)
 		)
@@
 	(wire
 		(pts
+			(xy 92.71 39.37) (xy 138.43 39.37)
+		)
+		(stroke
+			(width 0)
+			(type default)
+		)
+	)
+	(wire
+		(pts
 			(xy 97.79 135.89) (xy 97.79 140.97)
 		)
@@
 			(width 0)
 			(type default)
+		)
+	)
+	(wire
+		(pts
+			(xy 92.71 39.37) (xy 92.71 41.91)
+		)
+		(stroke
+			(width 0)
+			(type default)
+		)
+	)
+	(label "LAMP_L_N"
+		(at 92.71 41.91 270)
+		(effects
+			(font
+				(size 1.27 1.27)
+			)
+			(justify right bottom)
+		)
+	)
+	(label "LAMP_R_N"
+		(at 119.38 113.03 90)
+		(effects
+			(font
+				(size 1.27 1.27)
+			)
+			(justify left bottom)
 		)
 	)
@@
 			)
 		)
-		(property "Value" "Conn_01x04"
+		(property "Value" "IND_OUTPUT"
 			(at 146.05 41.9099 0)
 			(show_name no)
