File: schematics/indicators_input.kicad_sch (KiCad schematic)
At the start: 8 parts, among them J8 Conn_01x03_Pin, U4 SRV05-4

Commit message: schematics: Add mounting points for the PCB
Parts:
- J8: value Conn_01x03_Pin -> IND_INPUT
Changed lines of the file:
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@@
 			)
 		)
-		(property "Value" "Conn_01x03_Pin"
+		(property "Value" "IND_INPUT"
 			(at 74.295 82.55 0)
 			(show_name no)
