File: schematics/power.kicad_sch (KiCad schematic)
At the start: 10 parts, among them J3 Conn_01x02_Pin, U2 TSR2-2450

Commit message: kicad: Run Assign footprint
Parts:
- C2: footprint (none) -> Capacitor_SMD:C_1206_3216Metric
- C3: footprint (none) -> Capacitor_SMD:CP_Elec_6.3x7.7
- C4: footprint (none) -> Capacitor_SMD:C_0805_2012Metric
- F1, F2: footprint (none) -> Fuse:Fuse_1812_4532Metric
- J3: footprint (none) -> Connector_JST:JST_VH_B2P-VH-B_1x02_P3.96mm_Vertical
Changed lines of the file:
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@@
 			)
 		)
-		(property "Footprint" ""
+		(property "Footprint" "Capacitor_SMD:C_0805_2012Metric"
 			(at 185.1152 130.81 0)
 			(hide yes)
@@
 			)
 		)
-		(property "Footprint" ""
+		(property "Footprint" "Fuse:Fuse_1812_4532Metric"
 			(at 104.14 114.3 0)
 			(hide yes)
@@
 			)
 		)
-		(property "Footprint" ""
+		(property "Footprint" "Capacitor_SMD:CP_Elec_6.3x7.7"
 			(at 157.1752 130.81 0)
 			(hide yes)
@@
 			)
 		)
-		(property "Footprint" ""
+		(property "Footprint" "Fuse:Fuse_1812_4532Metric"
 			(at 76.2 73.66 0)
 			(hide yes)
@@
 			)
 		)
-		(property "Footprint" ""
+		(property "Footprint" "Capacitor_SMD:C_1206_3216Metric"
 			(at 147.0152 134.62 0)
 			(hide yes)
@@
 			)
 		)
-		(property "Footprint" ""
+		(property "Footprint" "Connector_JST:JST_VH_B2P-VH-B_1x02_P3.96mm_Vertical"
 			(at 34.29 135.89 0)
 			(hide yes)

Commit message: schematics: Add mounting points for the PCB
Parts:
- J3: value Conn_01x02_Pin -> POWER
Connections:
- net 5V_PRE: now reaches C4.1, D4.2 (A), U2.3 (Vout)
- net VIN_RAW: now reaches F1.1, F2.1, J3.1 (Pin_1)
- net VIN_RAW: no longer D2.2 (A), F1.2
- new net VIN_FUSED: D2.2 (A), F1.2
Changed lines of the file:
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@@
+	)
+	(junction
+		(at 45.72 123.19)
+		(diameter 0)
+		(color 0 0 0 0)
+	)
+	(junction
+		(at 106.68 115.57)
+		(diameter 0)
+		(color 0 0 0 0)
 	)
 	(junction
@@
 	)
 	(junction
+		(at 189.23 115.57)
+		(diameter 0)
+		(color 0 0 0 0)
+	)
+	(junction
 		(at 116.84 115.57)
 		(diameter 0)
@@
 	)
 	(junction
-		(at 95.25 115.57)
-		(diameter 0)
-		(color 0 0 0 0)
-	)
-	(junction
 		(at 156.21 115.57)
-		(diameter 0)
-		(color 0 0 0 0)
-	)
-	(junction
-		(at 102.87 115.57)
 		(diameter 0)
 		(color 0 0 0 0)
@@
 	(wire
 		(pts
+			(xy 95.25 115.57) (xy 95.25 135.89)
+		)
+		(stroke
+			(width 0)
+			(type default)
+		)
+	)
+	(wire
+		(pts
 			(xy 152.4 152.4) (xy 152.4 161.29)
 		)
@@
 	(wire
 		(pts
-			(xy 45.72 74.93) (xy 45.72 135.89)
+			(xy 189.23 111.76) (xy 189.23 115.57)
+		)
+		(stroke
+			(width 0)
+			(type default)
+		)
+	)
+	(wire
+		(pts
+			(xy 45.72 74.93) (xy 45.72 123.19)
 		)
 		(stroke
@@
 	(wire
 		(pts
-			(xy 184.15 115.57) (xy 190.5 115.57)
+			(xy 184.15 115.57) (xy 189.23 115.57)
 		)
 		(stroke
@@
 	(wire
 		(pts
+			(xy 45.72 123.19) (xy 45.72 135.89)
+		)
+		(stroke
+			(width 0)
+			(type default)
+		)
+	)
+	(wire
+		(pts
+			(xy 189.23 115.57) (xy 190.5 115.57)
+		)
+		(stroke
+			(width 0)
+			(type default)
+		)
+	)
+	(wire
+		(pts
 			(xy 156.21 115.57) (xy 158.75 115.57)
 		)
@@
 	(wire
 		(pts
+			(xy 40.64 123.19) (xy 45.72 123.19)
+		)
+		(stroke
+			(width 0)
+			(type default)
+		)
+	)
+	(wire
+		(pts
+			(xy 106.68 105.41) (xy 106.68 115.57)
+		)
+		(stroke
+			(width 0)
+			(type default)
+		)
+	)
+	(wire
+		(pts
 			(xy 102.87 115.57) (xy 106.68 115.57)
 		)
@@
 		)
 	)
-	(wire
-		(pts
-			(xy 102.87 115.57) (xy 95.25 115.57)
-		)
-		(stroke
-			(width 0)
-			(type default)
-		)
-	)
-	(wire
-		(pts
-			(xy 95.25 135.89) (xy 95.25 115.57)
-		)
-		(stroke
-			(width 0)
-			(type default)
+	(label "VIN_RAW"
+		(at 40.64 123.19 180)
+		(effects
+			(font
+				(size 1.27 1.27)
+			)
+			(justify right bottom)
+		)
+	)
+	(label "VIN_FUSED"
+		(at 106.68 105.41 90)
+		(effects
+			(font
+				(size 1.27 1.27)
+			)
+			(justify left bottom)
+		)
+	)
+	(label "5V_PRE"
+		(at 189.23 111.76 90)
+		(effects
+			(font
+				(size 1.27 1.27)
+			)
+			(justify left bottom)
 		)
 	)
@@
 			)
 		)
-		(property "Value" "Conn_01x02_Pin"
+		(property "Value" "POWER"
 			(at 34.925 133.35 0)
 			(show_name no)
